File: hardware/pcbs/OuchButtonV2/OuchButtonV2.kicad_pcb (KiCad board)
At the start: 4 copper layers, 78 parts, among them J1 USB_C_Receptacle_USB2.0_14P, J3 Conn_01x01_Pin, Q1 AO3423 P-Chanel, U1 ESP32-C6-MINI-1/U, U2 RT9080-33GJ5, U3 MCP73831-2-OT, U4 MPU-6050, U5 DS1307Z+, U6 AT42QT1010-TSHR, U7 TS3A24159DGS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

Commit message: Half done pcb
Parts:
- C1, C10, C11, C12, C13, C14, C15, C16, C17, C18, C2, C3, C4, C5, C6, C7, C8, C9: footprint Capacitor_SMD:C_0603_1608Metric_Pad1.08x0.95mm_HandSolder -> Capacitor_SMD:C_0805_2012Metric
- D1: footprint Diode_SMD:D_0603_1608Metric_Pad1.05x0.95mm_HandSolder -> Diode_SMD:D_0805_2012Metric
- D2: footprint LED_SMD:LED_0603_1608Metric_Pad1.05x0.95mm_HandSolder -> LED_SMD:LED_0805_2012Metric
- R1, R10, R11, R12, R13, R14, R15, R16, R17, R18, R2, R3, R4, R5, R6, R7, R9: footprint Resistor_SMD:R_0603_1608Metric_Pad0.98x0.95mm_HandSolder -> Resistor_SMD:R_0805_2012Metric
- R19, R20, R8: footprint Resistor_SMD:R_0603_1608Metric_Pad0.98x0.95mm_HandSolder -> Capacitor_SMD:C_0805_2012Metric
- moved D1 139.3 mm to (62.2, 41.3), turned to 0 degrees
- moved C5 137.8 mm to (54.8, 41.3)
- moved Q1 134.9 mm to (62.4, 38.1)
- moved C1 133.2 mm to (51.0, 44.6), turned to -90 degrees
- moved R4 131.6 mm to (81.3, 42.0), turned to 90 degrees
- moved C2 130.5 mm to (75.7, 45.2)
- moved U2 129.2 mm to (54.7, 44.6)
- moved U3 126.8 mm to (77.8, 42.0)
- moved R5 123.9 mm to (74.3, 42.0), turned to -90 degrees
- moved C3 116.0 mm to (79.9, 45.2), turned to 0 degrees
- moved R3 110.7 mm to (58.6, 44.6), turned to 90 degrees
- moved R7 108.7 mm to (197.1, 181.8), turned to 90 degrees
- moved R8 103.5 mm to (61.2, 44.6), turned to -90 degrees
- moved R6 97.3 mm to (194.7, 181.8), turned to -90 degrees
- moved U4 85.5 mm to (106.7, 86.8), turned to -90 degrees
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Connections:
- U1 pad 20: IO15/TOUCH -> unconnected-(U1-GPIO15-Pad20)
- U1 pad 29: IO23/AFE_RST -> IO23/TOUCH
- U6 pad 1: IO15/TOUCH -> IO23/TOUCH
Routing:
- net IO23/TOUCH: track 0.00 -> 29.2 mm, vias 0 -> 1
- net IO6/SDA: track 0.00 -> 29.1 mm, vias 0 -> 1
- net IO7/SCL: track 0.00 -> 28.9 mm, vias 0 -> 1
- net Net-(D1-K): track 0.00 -> 13.2 mm
- net Net-(U6-SNSK): track 0.00 -> 5.18 mm
- net Net-(JP8-C): track 0.00 -> 5.15 mm
- net Net-(U5-X2): track 0.00 -> 5.10 mm
- net Net-(D5-DOUT): track 0.00 -> 3.17 mm
- net Net-(D4-DOUT): track 0.00 -> 3.17 mm
- net Net-(D3-DOUT): track 0.00 -> 3.17 mm
- net Net-(U2-EN): track 0.00 -> 2.56 mm
- net Net-(J3-Pin_1): track 0.00 -> 2.42 mm
- net Net-(U6-SNS): track 0.00 -> 2.41 mm
- net IO2/BATT: track 0.00 -> 2.36 mm
- net IO3/CHG: track 0.00 -> 2.36 mm
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Other:
- board outline added: 42 x 41.5 mm

Commit message: Ready for review pcb
Parts:
- removed the D2 at (36.6, 169.2)
- removed JP1, JP2: SolderJumper_2_Bridged, Jumper:SolderJumper-2_P1.3mm_Open_RoundedPad1.0x1.5mm
- removed JP7: SolderJumper_3_Bridged123, Jumper:SolderJumper-3_P1.3mm_Open_RoundedPad1.0x1.5mm_NumberLabels
- R18: moved to B.Cu
- R19, R20: moved to F.Cu
- U7: footprint Package_CSP:LFCSP-16-1EP_4x4mm_P0.65mm_EP2.1x2.1mm -> Package_SO:TSSOP-10_3x3mm_P0.5mm
- moved R7 148.8 mm to (80.2, 89.6), turned to -90 degrees
- moved R6 145.4 mm to (82.3, 89.6), turned to 90 degrees
- moved U7 88.4 mm to (100.6, 91.7)
- moved U9 86.5 mm to (111.6, 95.0), turned to -90 degrees
- moved TP3 82.5 mm to (100.2, 83.2)
- moved FL1 78.8 mm to (105.4, 91.3), turned to -90 degrees
- moved TP2 77.2 mm to (110.6, 89.2)
- moved R21 68.3 mm to (95.4, 80.4), turned to 90 degrees
- moved TP4 67.4 mm to (96.5, 100.9)
- moved D2 65.0 mm to (97.5, 80.4), turned to 90 degrees
- moved TP1 64.8 mm to (110.5, 99.8)
- moved C10 64.7 mm to (87.3, 93.7)
- moved C17 64.6 mm to (91.0, 99.6), turned to 0 degrees
- moved R13 63.7 mm to (78.9, 93.2)
- moved R17 60.4 mm to (113.2, 90.0), turned to -90 degrees
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Connections:
- J1 pad A6: Net-(JP2-B) -> Net-(J1-D+-PadA6)
- J1 pad A7: Net-(JP1-A) -> Net-(J1-D--PadA7)
- J1 pad B6: Net-(JP2-A) -> Net-(J1-D+-PadA6)
- J1 pad B7: Net-(JP1-B) -> Net-(J1-D--PadA7)
- MK1 pad 6: IO21/SD -> IO14/SD
- R10 pad 1: IO6/SDA -> +3V3
- R10 pad 2: Net-(JP7-A) -> IO6/SDA
- R12 pad 2: IO14/S1 -> IO21/S1
- R17 pad 2: IO23/AFE_RST -> IO15/AFE_RST
- R18 pad 1: IO21/SD -> IO14/SD
- R19 pad 2: Net-(JP1-B) -> Net-(J1-D--PadA7)
- R20 pad 2: Net-(JP2-B) -> Net-(J1-D+-PadA6)
- R9 pad 1: Net-(JP7-B) -> +3V3
- S1 pad 2: IO14/S1 -> IO21/S1
- U1 pad 19: IO14/S1 -> IO14/SD
- U1 pad 20: unconnected-(U1-GPIO15-Pad20) -> IO15/AFE_RST
- U1 pad 27: IO21/SD -> IO21/S1
- U8 pad D1: IO23/AFE_RST -> IO15/AFE_RST
Routing:
- net +3V3: track 2.35 -> 59.7 mm, vias 0 -> 17
- net IO4/WB2812B: track 0.00 -> 42.0 mm
- net IO15/AFE_RST: track 0.00 -> 41.9 mm, vias 0 -> 3
- net VBATT: track 2.25 -> 39.0 mm, vias 0 -> 1
- net IO21/S1: track 0.00 -> 35.5 mm, vias 0 -> 2
- net EN: track 0.00 -> 32.0 mm, vias 0 -> 1
- net VCC_TX: track 0.00 -> 31.7 mm, vias 0 -> 2
- net VUSB: track 2.25 -> 34.0 mm, vias 0 -> 1
- net IO3/CHG: track 2.36 -> 32.8 mm, vias 0 -> 1
- net IO6/SDA: track 29.1 -> 58.2 mm, vias 1 -> 5
- net IO7/SCL: track 28.9 -> 57.7 mm, vias 1 -> 3
- net IO5/SELECT: track 0.00 -> 27.8 mm, vias 0 -> 3
- net IO9/BOOT: track 0.00 -> 27.7 mm
- net TX1: track 0.00 -> 26.7 mm, vias 0 -> 2
- net Net-(U8-CLK): track 0.00 -> 23.9 mm, vias 0 -> 2
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- added copper zone on In1.Cu, net +3V3
- added copper zone on B.Cu, net GND
- added copper zone on F.Cu, net GND
- added copper zone on In2.Cu, net GND
Other:
- board text added: "EAT40006 FYP"
- board text added: "V2.0 Ouch Button"
- board text added: "x"
- board text added: "y"
