File: hardware/pcbs/OuchButtonV2/OuchButtonV2.kicad_sch (KiCad schematic)
At the start: 4 parts, among them J1 USB_C_Receptacle_USB2.0_14P, U1 ESP32-C6-MINI-1/U, U2 RT9080-33GJ5

Commit message: Finished schematic
Parts:
- removed D1: LED, symbol Device:LED
- added BOOT, RST: SW_Push, Button_Switch_SMD:SW_SPST_CK_RS282G05A3, symbol Switch:SW_Push
- added C1, C2, C5: 2.2uF, symbol Device:C_Small
- added C10, C11, C12, C13, C16, C17, C6, C8: 0.1uF, Capacitor_SMD:C_0603_1608Metric_Pad1.08x0.95mm_HandSolder, symbol Device:C_Small
- added C14, C15: 1uF, Capacitor_SMD:C_0603_1608Metric_Pad1.08x0.95mm_HandSolder, symbol Device:C_Small
- added C18: 22uF, Capacitor_SMD:C_0603_1608Metric_Pad1.08x0.95mm_HandSolder, symbol Device:C_Small
- added C3, C4: 2.2uF, Capacitor_SMD:C_0603_1608Metric_Pad1.08x0.95mm_HandSolder, symbol Device:C_Small
- added C7: 2.2nF, Capacitor_SMD:C_0603_1608Metric_Pad1.08x0.95mm_HandSolder, symbol Device:C_Small
- added C9: 10nF, Capacitor_SMD:C_0603_1608Metric_Pad1.08x0.95mm_HandSolder, symbol Device:C_Small
- added D1: 5V Min, Diode_SMD:D_0603_1608Metric_Pad1.05x0.95mm_HandSolder, symbol Device:D_Schottky
- added D2: Red, LED_SMD:LED_0603_1608Metric_Pad1.05x0.95mm_HandSolder, symbol Device:LED
- added D3: WS2812B, LED_SMD:LED_WS2812B-2020_PLCC4_2.0x2.0mm, symbol LED:WS2812B-2020
- added D4, D5, D6: WS2812B-2020, LED_SMD:LED_WS2812B-2020_PLCC4_2.0x2.0mm, symbol LED:WS2812B-2020
- added FL1: 0603USB-951, Inductor_SMD:L_CommonMode_Wurth_WE-CNSW-1206, symbol Filter:Choke_Coilcraft_0603USB-951
- added J2: Solder with Relief, Connector_Wire:SolderWire-1.5sqmm_1x02_P7.8mm_D1.7mm_OD3.9mm_Relief, symbol Connector:Conn_01x02_Socket
- added J3: Conn_01x01_Pin, Connector_Wire:SolderWire-0.5sqmm_1x01_D0.9mm_OD2.1mm, symbol Connector:Conn_01x01_Pin
- added JP1, JP2, JP4, JP5, SHLD: SolderJumper_2_Bridged, symbol Jumper:SolderJumper_2_Bridged
- added JP3, JP8: SolderJumper_3_Bridged12, symbol Jumper:SolderJumper_3_Bridged12
- added JP7: SolderJumper_3_Bridged123, symbol Jumper:SolderJumper_3_Bridged123
- added LED1: SFH 7072, SFH_7072:SFH 7072_OSR, symbol SFH_7072:SFH_7072
- added MK1: ICS-43434, Sensor_Audio:InvenSense_ICS-43434-6_3.5x2.65mm, symbol Sensor_Audio:ICS-43434
- added Q1: PMOS, symbol Simulation_SPICE:PMOS
- added R1, R2: 5.1k, Resistor_SMD:R_0603_1608Metric_Pad0.98x0.95mm_HandSolder, symbol Device:R_Small
- added R10, R16, R17, R4, R5, R9: 4.7k, Resistor_SMD:R_0603_1608Metric_Pad0.98x0.95mm_HandSolder, symbol Device:R_Small
- added R11, R12, R13, R18, R3, R8: 100k, Resistor_SMD:R_0603_1608Metric_Pad0.98x0.95mm_HandSolder, symbol Device:R_Small
- added R14: 10k, Resistor_SMD:R_0603_1608Metric_Pad0.98x0.95mm_HandSolder, symbol Device:R_Small
- added R15: 470, Resistor_SMD:R_0603_1608Metric_Pad0.98x0.95mm_HandSolder, symbol Device:R_Small
- added R19, R20: 22R, Resistor_SMD:R_0603_1608Metric_Pad0.98x0.95mm_HandSolder, symbol Device:R_Small
- added R6, R7: 10M, Resistor_SMD:R_0603_1608Metric_Pad0.98x0.95mm_HandSolder, symbol Device:R_Small
- added S1: SW_Push, Button_Switch_SMD:SW_SPST_CK_KMS2xxGP, symbol Switch:SW_Push
- added TP1/3.3V, TP2/SDA, TP3/SCL, TP4/GND: TestPoint, TestPoint:TestPoint_Pad_D1.0mm, symbol Connector:TestPoint
- added U3: MCP73831-2-OT, Package_TO_SOT_SMD:SOT-23-5, symbol Battery_Management:MCP73831-2-OT
- added U4: MPU-6050, Sensor_Motion:InvenSense_QFN-24_4x4mm_P0.5mm, symbol Sensor_Motion:MPU-6050
- added U5: DS1307Z+, Package_SO:SOIC-8_3.9x4.9mm_P1.27mm, symbol Timer_RTC:DS1307Z+
- added U6: AT42QT1010-TSHR, Package_TO_SOT_SMD:SOT-23-6, symbol Sensor_Touch:AT42QT1010-TSHR
- added U7: TS3A24159DGS, Package_CSP:LFCSP-16-1EP_4x4mm_P0.65mm_EP2.1x2.1mm, symbol Analog_Switch:TS3A24159DGS
- added U8: AFE4404YZPT, AFE4404YZPT:YZP15_TEX, symbol AFE4404YZPT:AFE4404YZPT
- added U9: WE-TVS-82400102, Package_TO_SOT_SMD:SOT-23-6, symbol Power_Protection:WE-TVS-82400102
- added Y1: 32.768 kHz, Crystal:Crystal_SMD_2012-2Pin_2.0x1.2mm_HandSoldering, symbol Device:Crystal
- U2: footprint TSOT-23-5_RIT -> RT9080:TSOT-23-5_RIT
Connections:
- net +3V3: now also C12.1, C15.1, C16.1, C17.1, C18.1, C8.1, C9.1, JP3.3 (B), JP7.2 (C), JP8.3 (B), MK1.5 (VDD), R11.1, R12.1, R13.1, R17.1, TP1/3.3V.1, U4.13 (VDD), U4.8 (VLOGIC), U5.8 (VCC), U6.5 (VDD), U7.1 (VCC), U8.A2 (RX_SUP), U8.A3 (IO_SUP), U9.5
- net GND: now also J1.A1 (GND), J1.A12 (GND), J1.B1 (GND), J1.B12 (GND), U2.2 (GND), BOOT.1, C1.2, C10.2, C12.2, C13.2, C14.2, C15.2, C16.2, C17.2, C18.2, C2.2, C3.2, C4.2, C5.2, C6.2, C7.2, C8.2, C9.2, D3.2 (VSS), D4.2 (VSS), D5.2 (VSS), D6.2 (VSS), J2.2 (Pin_2), JP3.1 (A), JP4.1 (A), JP5.1 (A), JP8.1 (A), MK1.3 (GND), R1.2, R16.2, R18.2, R2.2, R5.2, R6.2, R8.2, RST.1, S1.1, SHLD.1 (A), TP4/GND.1, U3.2 (V_{SS}), U4.18 (GND), U5.4 (GND), U6.2 (VSS), U6.6 (SYNC), U7.6 (GND), U8.D3 (GND), U9.2
- net at U2.1 (VIN): now also C5.1, D1.1 (K), Q1.3 (S), R3.2, R8.1
- net at U2.3 (EN): now also R3.1
- net +3.3V: now reaches U2.5 (VOUT)
- net +3.3V: now also C1.1
- net VUSB: now reaches J1.A4 (VBUS), J1.A9 (VBUS), J1.B4 (VBUS), J1.B9 (VBUS)
- net VUSB: now also C2.1, D1.2 (A), Q1.2 (G), R4.1, U3.4 (V_{DD})
- net at J1.A5 (CC1): now also R2.1
- net at J1.A6 (D+): now also JP2.2 (B), R20.2
- net at J1.A7 (D-): now also JP1.1 (A)
- net at J1.B5 (CC2): now also R1.1
- net at J1.B6 (D+): now also JP2.1 (A)
- net at J1.B7 (D-): now also JP1.2 (B), R19.2
- net at J1.S1 (SHIELD): now also SHLD.2 (B)
- net IO5/SELECT: now reaches U1.10 (MTDI/GPIO5/ADC1_CH5)
- net IO5/SELECT: now also U7.4, U7.8
- net IO6/SDA: now reaches U1.15 (MTCK/GPIO6/ADC1_CH6)
- net IO6/SDA: now also R10.1, TP2/SDA.1, U4.24 (SDA), U5.6 (SCL), U8.E2 (I2C_CLK)
- net IO7/SCL: now reaches U1.16 (MTDO/GPIO7)
- net IO7/SCL: now also R9.2, TP3/SCL.1, U4.23 (SCL), U5.5 (SDA), U8.E1 (I2C_DAT)
- net IO14/S1: now reaches U1.19 (GPIO14)
- net IO14/S1: now also R12.2, S1.2
- net IO15/TOUCH: now reaches U1.20 (GPIO15)
- net IO15/TOUCH: now also U6.1 (OUT)
- net at U1.22 (GPIO8): now also R13.2
- net IO9/BOOT: now reaches U1.23 (GPIO9)
- net IO9/BOOT: now also BOOT.2
- net IO18/LR: now reaches U1.24 (GPIO18)
- net IO18/LR: now also MK1.2 (LR)
- net IO19/WS: now reaches U1.25 (GPIO19)
- net IO19/WS: now also MK1.1 (WS)
- net IO20/SCK: now reaches U1.26 (GPIO20)
- net IO20/SCK: now also MK1.4 (SCK)
- net IO21/SD: now reaches U1.27 (GPIO21)
- net IO21/SD: now also MK1.6 (SD), R18.1
- net IO22/AFE_CLK: now reaches U1.28 (GPIO22)
- net IO22/AFE_CLK: now also R15.2, R16.1
- net IO23/AFE_RST: now reaches U1.29 (GPIO23)
- net IO23/AFE_RST: now also R17.2, U8.D1 (RESETZ)
- net IO2/BATT: now reaches U1.5 (GPIO2/ADC1_CH2)
- net IO2/BATT: now also C4.1, R6.1, R7.2
- net IO3/WB2812B: now reaches U1.6 (GPIO3/ADC1_CH3)
- net IO3/WB2812B: now also D3.3 (DIN)
- net EN: now reaches U1.8 (EN/CHIP_PU)
- net EN: now also C10.1, R11.2, RST.2
- net USB_D+ renamed IO13/USB_D+
- net IO13/USB_D+: now also R20.1
- net USB_D- renamed IO12/USB_D-
- net IO12/USB_D-: now also R19.1
- new net: JP7.3 (B), R9.1
- new net: FL1.2, U8.A1 (INM)
- new net: FL1.3, U8.B1 (INP)
- new net: R15.1, U8.C2 (CLK)
- new net: JP7.1 (A), R10.2
- new net: D5.1 (DOUT), D6.3 (DIN)
- new net: D2.1 (K), U3.1 (STAT)
- new net: D2.2 (A), R4.2
- new net: JP3.2 (C), U4.9 (AD0)
- new net: FL1.1, U7.9
- new net: FL1.4, U7.3
- new net: R5.1, U3.5 (PROG)
- new net: U5.1 (X1), Y1.1
- new net: U5.2 (X2), Y1.2
- new net: JP8.2 (C), U5.3 (VBAT)
- new net: C7.1, U4.20 (CPOUT)
- new net: C11.1, R14.2, U6.3 (SNSK)
- new net: C11.2, U6.4 (SNS)
- new net: J3.1 (Pin_1), R14.1
- new net: JP4.2 (B), U4.1 (CLKIN)
- new net: D4.1 (DOUT), D5.3 (DIN)
- new net: D3.1 (DOUT), D4.3 (DIN)
- new net: C6.1, U4.10 (REGOUT)
- new net: JP5.2 (B), U4.11 (FSYNC)
- new net INM1: LED1.10 (IPA), U7.7
- new net INM2: LED1.2 (BPA), U7.10
- new net INP1: LED1.3 (IPC), U7.5
- new net INP2: LED1.1 (BPC), U7.2
- new net TX1: LED1.12 (G2C), LED1.6 (G1C), U8.B3 (TX1)
- new net TX2: LED1.8 (RC), U8.D2 (TX2)
- new net TX3: LED1.9 (IC), U8.C3 (TX3)
- new net VBATT: C3.1, D3.4 (VDD), D4.4 (VDD), D5.4 (VDD), D6.4 (VDD), J2.1 (Pin_1), Q1.1 (D), R7.1, U3.3 (V_{BAT})
- new net VCC_TX: C13.1, C14.1, LED1.11 (G2A), LED1.4 (IA), LED1.5 (G1A), LED1.7 (RA), U8.E3 (TX_SUP)
- no-connect marks 0 -> 5
Other:
- note added: "3.3V Regulator"
- note added: "ADO High -> I2C addr: b1101000 ADO Low -> I2C addr: b1101001"
- note added: "Battery Charger"
- note added: "Battery Voltage"
- note added: "Buttons"
- note added: "Capacitive Touch"
- note added: "ESD Protection"
- note added: "HRM and SPO2 Sensor"
- note added: "Hot swappable with TTP223-BA6"
- note added: "I2C Pullups"
- note added: "IMU"
- note added: "I_CHG = 1000/R_PROG = 1000/4.7k = 213mA"
- note added: "MCU: ESP32-C6"
- note added: "MEMS Microphone"
- note added: "Max Input Voltage: 5.5V Max Current: 600mA"
- note added: "RTC"
- note added: "Rs: 1kΩ -> 10kΩ Cs: 1nF -> 47nF"
- note added: "Test Points"
- note added: "Touch pad is off the PCB"
- note added: "USB-C Connector"
- note added: "WS2812B-2020 LEDs"
- moved on the sheet: J1, U1

Commit message: Start PCB layout
Parts:
- removed BOOT, RST: SW_Push, Button_Switch_SMD:SW_SPST_CK_RS282G05A3, symbol Switch:SW_Push
- added BOOT1, RST1: SolderJumper_2_Open, Jumper:SolderJumper-2_P1.3mm_Open_RoundedPad1.0x1.5mm, symbol Jumper:SolderJumper_2_Open
- added R21: 4.7k, Resistor_SMD:R_0603_1608Metric_Pad0.98x0.95mm_HandSolder, symbol Device:R_Small
- C1, C2, C5: footprint (none) -> Capacitor_SMD:C_0603_1608Metric_Pad1.08x0.95mm_HandSolder
- D2: value Red -> LED
- J1: footprint (none) -> Connector_USB:USB_C_Receptacle_G-Switch_GT-USB-7025
- J3: footprint Connector_Wire:SolderWire-0.5sqmm_1x01_D0.9mm_OD2.1mm -> Connector_Wire:SolderWirePad_1x01_SMD_1x2mm
- JP1, JP2, JP4, JP5: footprint (none) -> Jumper:SolderJumper-2_P1.3mm_Open_RoundedPad1.0x1.5mm
- JP3, JP7, JP8: footprint (none) -> Jumper:SolderJumper-3_P1.3mm_Open_RoundedPad1.0x1.5mm_NumberLabels
- J_BATT1: renamed from J2; footprint Connector_Wire:SolderWire-1.5sqmm_1x02_P7.8mm_D1.7mm_OD3.9mm_Relief -> Connector_Wire:SolderWire-0.1sqmm_1x02_P3.6mm_D0.4mm_OD1mm
- Q1: value PMOS -> AO3423 P-Chanel; footprint (none) -> Package_TO_SOT_SMD:SOT-23-3
- R4: value 4.7k -> 10k
- SHLD1: renamed from SHLD; footprint (none) -> Jumper:SolderJumper-2_P1.3mm_Open_RoundedPad1.0x1.5mm
- U2: footprint RT9080:TSOT-23-5_RIT -> RT9080_33GJ5:TSOT-23-5_RIT
- renumbered TP1/3.3V to TP1, TP2/SDA to TP2, TP3/SCL to TP3, TP4/GND to TP4
Connections:
- net +3.3V is gone; now on net +3V3: C1.1, U2.5 (VOUT)
- net +3V3: now also R4.1
- net EN: now also RST1.2 (B)
- net GND: now also D2.1 (K), BOOT1.1 (A), RST1.1 (A)
- net IO9/BOOT: now also BOOT1.2 (B)
- net VUSB: now also R21.1; no longer R4.1
- net IO3/CHG: now reaches U3.1 (STAT)
- net IO3/CHG: now also R4.2, U1.6 (GPIO3/ADC1_CH3); no longer D2.1 (K)
- net at D2.2 (A): now also R21.2; no longer R4.2
- net IO4/WB2812B: now reaches U1.9 (MTMS/GPIO4/ADC1_CH4)
- net IO4/WB2812B: now also D3.3 (DIN)
- removed net IO3/WB2812B: D3.3 (DIN), U1.6 (GPIO3/ADC1_CH3)
Other:
- note added: "Power LEDs"
- title: Microcontroller -> Main
- moved on the sheet: C10, R4, U9

Commit message: Half done pcb
Parts:
- C1, C10, C11, C12, C13, C14, C15, C16, C17, C18, C2, C3, C4, C5, C6, C7, C8, C9: footprint Capacitor_SMD:C_0603_1608Metric_Pad1.08x0.95mm_HandSolder -> Capacitor_SMD:C_0805_2012Metric
- D1: footprint Diode_SMD:D_0603_1608Metric_Pad1.05x0.95mm_HandSolder -> Diode_SMD:D_0805_2012Metric
- D2: footprint LED_SMD:LED_0603_1608Metric_Pad1.05x0.95mm_HandSolder -> LED_SMD:LED_0805_2012Metric
- R1, R10, R11, R12, R13, R14, R15, R16, R17, R18, R2, R3, R4, R5, R6, R7, R9: footprint Resistor_SMD:R_0603_1608Metric_Pad0.98x0.95mm_HandSolder -> Resistor_SMD:R_0805_2012Metric
- R19, R20, R8: footprint Resistor_SMD:R_0603_1608Metric_Pad0.98x0.95mm_HandSolder -> Capacitor_SMD:C_0805_2012Metric
Connections:
- net IO23/AFE_RST: no longer U1.29 (GPIO23)
- net IO15/TOUCH: no longer names the net of U1.20 (GPIO15)
- net IO15/TOUCH: no longer U6.1 (OUT)
- new net IO23/TOUCH: U1.29 (GPIO23), U6.1 (OUT)
Changed lines of the file:
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@@
 	(wire
 		(pts
-			(xy 91.44 232.41) (xy 97.79 232.41)
-		)
-		(stroke
-			(width 0)
-			(type default)
-		)
-	)
-	(wire
-		(pts
 			(xy 187.96 254) (xy 191.77 254)
 		)
@@
 	(wire
 		(pts
+			(xy 91.44 247.65) (xy 97.79 247.65)
+		)
+		(stroke
+			(width 0)
+			(type default)
+		)
+	)
+	(wire
+		(pts
 			(xy 241.3 264.16) (xy 252.73 264.16)
 		)
@@
 	(wire
 		(pts
-			(xy 91.44 247.65) (xy 97.79 247.65)
-		)
-		(stroke
-			(width 0)
-			(type default)
-		)
-	)
-	(wire
-		(pts
 			(xy 201.93 63.5) (xy 201.93 69.85)
 		)
@@
 		)
 	)
-	(global_label "IO15{slash}TOUCH"
+	(global_label "IO23{slash}TOUCH"
 		(shape input)
-		(at 97.79 232.41 0)
+		(at 97.79 247.65 0)
 		(fields_autoplaced yes)
 		(effects
@@
 		)
 		(property "Intersheetrefs" "${INTERSHEET_REFS}"
-			(at 112.6891 232.41 0)
+			(at 112.6891 247.65 0)
 			(effects
 				(font
@@
 		)
 	)
-	(global_label "IO15{slash}TOUCH"
+	(global_label "IO23{slash}TOUCH"
 		(shape input)
 		(at 237.49 203.2 180)
@@
 	(global_label "IO23{slash}AFE_RST"
 		(shape input)
-		(at 97.79 247.65 0)
+		(at 106.68 250.19 0)
 		(fields_autoplaced yes)
 		(effects
@@
 		)
 		(property "Intersheetrefs" "${INTERSHEET_REFS}"
-			(at 114.2009 247.65 0)
+			(at 123.0909 250.19 0)
 			(effects
 				(font
@@
 			)
 		)
-		(property "Footprint" "Resistor_SMD:R_0603_1608Metric_Pad0.98x0.95mm_HandSolder"
+		(property "Footprint" "Resistor_SMD:R_0805_2012Metric"
 			(at 151.13 207.01 0)
 			(effects
@@
 			)
 		)
-		(property "Footprint" "Resistor_SMD:R_0603_1608Metric_Pad0.98x0.95mm_HandSolder"
+		(property "Footprint" "Resistor_SMD:R_0805_2012Metric"
 			(at 160.02 247.65 0)
 			(effects
@@
 			)
 		)
-		(property "Footprint" "Resistor_SMD:R_0603_1608Metric_Pad0.98x0.95mm_HandSolder"
+		(property "Footprint" "Resistor_SMD:R_0805_2012Metric"
 			(at 383.54 128.27 0)
 			(effects
@@
 			)
 		)
-		(property "Footprint" "Capacitor_SMD:C_0603_1608Metric_Pad1.08x0.95mm_HandSolder"
+		(property "Footprint" "Capacitor_SMD:C_0805_2012Metric"
 			(at 236.22 161.29 0)
 			(effects
@@
 			)
 		)
-		(property "Footprint" "Capacitor_SMD:C_0603_1608Metric_Pad1.08x0.95mm_HandSolder"
+		(property "Footprint" "Capacitor_SMD:C_0805_2012Metric"
 			(at 165.1 261.62 0)
 			(effects
@@
 			)
 		)
-		(property "Footprint" "Resistor_SMD:R_0603_1608Metric_Pad0.98x0.95mm_HandSolder"
+		(property "Footprint" "Resistor_SMD:R_0805_2012Metric"
 			(at 176.53 207.01 0)
 			(effects
@@
 			)
 		)
-		(property "Footprint" "Resistor_SMD:R_0603_1608Metric_Pad0.98x0.95mm_HandSolder"
+		(property "Footprint" "Resistor_SMD:R_0805_2012Metric"
 			(at 207.01 165.1 0)
 			(effects
@@
 			)
 		)
-		(property "Footprint" "Resistor_SMD:R_0603_1608Metric_Pad0.98x0.95mm_HandSolder"
+		(property "Footprint" "Resistor_SMD:R_0805_2012Metric"
 			(at 213.36 63.5 0)
 			(effects
@@
 			)
 		)
-		(property "Footprint" "Resistor_SMD:R_0603_1608Metric_Pad0.98x0.95mm_HandSolder"
+		(property "Footprint" "Resistor_SMD:R_0805_2012Metric"
 			(at 95.25 199.39 0)
 			(effects
@@
 			)
 		)
-		(property "Footprint" "Capacitor_SMD:C_0603_1608Metric_Pad1.08x0.95mm_HandSolder"
+		(property "Footprint" "Capacitor_SMD:C_0805_2012Metric"
 			(at 274.32 60.96 0)
 			(effects
@@
 			)
 		)
-		(property "Footprint" "LED_SMD:LED_0603_1608Metric_Pad1.05x0.95mm_HandSolder"
+		(property "Footprint" "LED_SMD:LED_0805_2012Metric"
 			(at 370.84 231.14 0)
 			(effects
@@
 			)
 		)
-		(property "Footprint" "Capacitor_SMD:C_0603_1608Metric_Pad1.08x0.95mm_HandSolder"
+		(property "Footprint" "Capacitor_SMD:C_0805_2012Metric"
 			(at 105.41 143.51 0)
 			(effects
@@
 			)
 		)
-		(property "Footprint" "Capacitor_SMD:C_0603_1608Metric_Pad1.08x0.95mm_HandSolder"
+		(property "Footprint" "Capacitor_SMD:C_0805_2012Metric"
 			(at 267.97 204.47 0)
 			(effects
@@
 			)
 		)
-		(property "Footprint" "Resistor_SMD:R_0603_1608Metric_Pad0.98x0.95mm_HandSolder"
+		(property "Footprint" "Capacitor_SMD:C_0805_2012Metric"
 			(at 58.42 40.64 0)
 			(effects
@@
 			)
 		)
-		(property "Footprint" "Resistor_SMD:R_0603_1608Metric_Pad0.98x0.95mm_HandSolder"
+		(property "Footprint" "Resistor_SMD:R_0805_2012Metric"
 			(at 280.67 199.39 0)
 			(effects
@@
 			)
 		)
-		(property "Footprint" "Capacitor_SMD:C_0603_1608Metric_Pad1.08x0.95mm_HandSolder"
+		(property "Footprint" "Capacitor_SMD:C_0805_2012Metric"
 			(at 173.99 43.18 0)
 			(effects
@@
 			)
 		)
-		(property "Footprint" "Capacitor_SMD:C_0603_1608Metric_Pad1.08x0.95mm_HandSolder"
+		(property "Footprint" "Capacitor_SMD:C_0805_2012Metric"
 			(at 110.49 267.97 0)
 			(effects
@@
 			)
 		)
-		(property "Footprint" "Resistor_SMD:R_0603_1608Metric_Pad0.98x0.95mm_HandSolder"
+		(property "Footprint" "Resistor_SMD:R_0805_2012Metric"
 			(at 285.75 40.64 0)
 			(effects
@@
 			)
 		)
-		(property "Footprint" "Resistor_SMD:R_0603_1608Metric_Pad0.98x0.95mm_HandSolder"
+		(property "Footprint" "Resistor_SMD:R_0805_2012Metric"
 			(at 191.77 247.65 0)
 			(effects
@@
 			)
 		)
-		(property "Footprint" "Capacitor_SMD:C_0603_1608Metric_Pad1.08x0.95mm_HandSolder"
+		(property "Footprint" "Capacitor_SMD:C_0805_2012Metric"
 			(at 383.54 173.99 0)
 			(effects
@@
 			)
 		)
-		(property "Footprint" "Capacitor_SMD:C_0603_1608Metric_Pad1.08x0.95mm_HandSolder"
+		(property "Footprint" "Capacitor_SMD:C_0805_2012Metric"
 			(at 152.4 52.07 0)
 			(effects
@@
 			)
 		)
-		(property "Footprint" "Resistor_SMD:R_0603_1608Metric_Pad0.98x0.95mm_HandSolder"
+		(property "Footprint" "Resistor_SMD:R_0805_2012Metric"
 			(at 373.38 135.89 0)
 			(effects
@@
 			)
 		)
-		(property "Footprint" "Capacitor_SMD:C_0603_1608Metric_Pad1.08x0.95mm_HandSolder"
+		(property "Footprint" "Capacitor_SMD:C_0805_2012Metric"
 			(at 116.84 143.51 0)
 			(effects
@@
 			)
 		)
-		(property "Footprint" "Resistor_SMD:R_0603_1608Metric_Pad0.98x0.95mm_HandSolder"
+		(property "Footprint" "Capacitor_SMD:C_0805_2012Metric"
 			(at 58.42 38.1 0)
 			(effects
@@
 			)
 		)
-		(property "Footprint" "Resistor_SMD:R_0603_1608Metric_Pad0.98x0.95mm_HandSolder"
+		(property "Footprint" "Resistor_SMD:R_0805_2012Metric"
 			(at 45.72 59.69 0)
 			(effects
@@
 			)
 		)
-		(property "Footprint" "Capacitor_SMD:C_0603_1608Metric_Pad1.08x0.95mm_HandSolder"
+		(property "Footprint" "Capacitor_SMD:C_0805_2012Metric"
 			(at 394.97 173.99 0)
 			(effects
@@
 			)
 		)
-		(property "Footprint" "Capacitor_SMD:C_0603_1608Metric_Pad1.08x0.95mm_HandSolder"
+		(property "Footprint" "Capacitor_SMD:C_0805_2012Metric"
 			(at 113.03 53.34 0)
 			(effects
@@
 			)
 		)
-		(property "Footprint" "Resistor_SMD:R_0603_1608Metric_Pad0.98x0.95mm_HandSolder"
+		(property "Footprint" "Resistor_SMD:R_0805_2012Metric"
 			(at 186.69 53.34 0)
 			(effects
@@
 			)
 		)
-		(property "Footprint" "Resistor_SMD:R_0603_1608Metric_Pad0.98x0.95mm_HandSolder"
+		(property "Footprint" "Resistor_SMD:R_0805_2012Metric"
 			(at 383.54 142.24 0)
 			(effects
@@
 			)
 		)
-		(property "Footprint" "Diode_SMD:D_0603_1608Metric_Pad1.05x0.95mm_HandSolder"
+		(property "Footprint" "Diode_SMD:D_0805_2012Metric"
 			(at 96.52 45.72 0)
 			(effects
@@
 			)
 		)
-		(property "Footprint" "Capacitor_SMD:C_0603_1608Metric_Pad1.08x0.95mm_HandSolder"
+		(property "Footprint" "Capacitor_SMD:C_0805_2012Metric"
 			(at 370.84 173.99 0)
 			(effects
@@
 			)
 		)
-		(property "Footprint" "Resistor_SMD:R_0603_1608Metric_Pad0.98x0.95mm_HandSolder"
+		(property "Footprint" "Capacitor_SMD:C_0805_2012Metric"
 			(at 102.87 53.34 0)
 			(effects
@@
 			)
 		)
-		(property "Footprint" "Resistor_SMD:R_0603_1608Metric_Pad0.98x0.95mm_HandSolder"
+		(property "Footprint" "Resistor_SMD:R_0805_2012Metric"
 			(at 125.73 49.53 0)
 			(effects
@@
 			)
 		)
-		(property "Footprint" "Resistor_SMD:R_0603_1608Metric_Pad0.98x0.95mm_HandSolder"
+		(property "Footprint" "Resistor_SMD:R_0805_2012Metric"
 			(at 285.75 60.96 0)
 			(effects
@@
 			)
 		)
-		(property "Footprint" "Capacitor_SMD:C_0603_1608Metric_Pad1.08x0.95mm_HandSolder"
+		(property "Footprint" "Capacitor_SMD:C_0805_2012Metric"
 			(at 223.52 63.5 0)
 			(effects
@@
 			)
 		)
-		(property "Footprint" "Resistor_SMD:R_0603_1608Metric_Pad0.98x0.95mm_HandSolder"
+		(property "Footprint" "Resistor_SMD:R_0805_2012Metric"
 			(at 54.61 59.69 0)
 			(effects
@@
 			)
 		)
-		(property "Footprint" "Capacitor_SMD:C_0603_1608Metric_Pad1.08x0.95mm_HandSolder"
+		(property "Footprint" "Capacitor_SMD:C_0805_2012Metric"
 			(at 214.63 212.09 0)
 			(effects
@@
 			)
 		)
-		(property "Footprint" "Capacitor_SMD:C_0603_1608Metric_Pad1.08x0.95mm_HandSolder"
+		(property "Footprint" "Capacitor_SMD:C_0805_2012Metric"
 			(at 127 143.51 0)
 			(effects
@@
 			)
 		)
-		(property "Footprint" "Capacitor_SMD:C_0603_1608Metric_Pad1.08x0.95mm_HandSolder"
+		(property "Footprint" "Capacitor_SMD:C_0805_2012Metric"
 			(at 93.98 143.51 0)
 			(effects
@@
 			)
 		)
-		(property "Footprint" "Capacitor_SMD:C_0603_1608Metric_Pad1.08x0.95mm_HandSolder"
+		(property "Footprint" "Capacitor_SMD:C_0805_2012Metric"
 			(at 99.06 267.97 0)
 			(effects

Commit message: Ready for review pcb
Parts:
- removed JP1, JP2: SolderJumper_2_Bridged, Jumper:SolderJumper-2_P1.3mm_Open_RoundedPad1.0x1.5mm, symbol Jumper:SolderJumper_2_Bridged
- removed JP7: SolderJumper_3_Bridged123, Jumper:SolderJumper-3_P1.3mm_Open_RoundedPad1.0x1.5mm_NumberLabels, symbol Jumper:SolderJumper_3_Bridged123
- U7: footprint Package_CSP:LFCSP-16-1EP_4x4mm_P0.65mm_EP2.1x2.1mm -> Package_SO:TSSOP-10_3x3mm_P0.5mm
Connections:
- net IO23/AFE_RST is gone; now on net IO15/AFE_RST: R17.2, U8.D1 (RESETZ)
- net +3V3: now also R10.1, R9.1
- net IO6/SDA: now also R10.2; no longer R10.1
- net at J1.A7 (D-): now also J1.B7 (D-), R19.2
- net at J1.A6 (D+), R20.2: now also J1.B6 (D+)
- net IO15/AFE_RST: now reaches U1.20 (GPIO15)
- net IO14/S1 renamed IO21/S1
- net IO21/S1: now also U1.27 (GPIO21); no longer U1.19 (GPIO14)
- net IO21/SD renamed IO14/SD
- net IO14/SD: now also U1.19 (GPIO14); no longer U1.27 (GPIO21)
Other:
- moved on the sheet: R10, R19, R20, R9

Commit message: For manufacturing
Parts:
- D1: footprint Diode_SMD:D_0805_2012Metric -> Diode_SMD:D_SOD-323
- FL1: value 0603USB-951 -> 744232090
Changed lines of the file:
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@@
 			)
 		)
-		(property "Value" "0603USB-951"
+		(property "Value" "744232090"
 			(at 324.739 110.49 0)
 			(effects
@@
 			)
 		)
-		(property "Datasheet" "https://www.coilcraft.com/pdfs/0603usb.pdf"
+		(property "Datasheet" "CMC 370MA 2LN 90OHM SMD AEC-Q200"
 			(at 325.12 123.825 0)
 			(effects
@@
 			)
 		)
-		(property "Footprint" "Diode_SMD:D_0805_2012Metric"
+		(property "Footprint" "Diode_SMD:D_SOD-323"
 			(at 96.52 45.72 0)
 			(effects
